Commit message: feat: b2 코드 정리

File: b2_description/urdf/b2_description.urdf (robot description, URDF)
Before this commit: robot b2_description, 37 links, 36 joints
Links:
- link FL_calf: geometry collision box size=0.05 0.028 0.035; collision box size=0.1 0.0245 0.018
- link FL_hip: geometry collision cylinder length=0.05 radius=0.07; visual mesh filename=package://b2_driver_description/meshes/FL_hip.dae
- link FL_thigh: geometry collision box size=0.32 0.0445 0.054; visual mesh filename=package://b2_driver_description/meshes/FL_thigh.dae
- link FR_calf: geometry collision box size=0.05 0.028 0.035; collision box size=0.1 0.0245 0.018
- link FR_hip: geometry collision cylinder length=0.05 radius=0.07; visual mesh filename=package://b2_driver_description/meshes/FR_hip.dae
- link FR_thigh: geometry collision box size=0.25 0.028 0.04; visual mesh filename=package://b2_driver_description/meshes/FR_thigh.dae
- link RL_calf: geometry collision box size=0.05 0.028 0.035; collision box size=0.1 0.0245 0.018
- link RL_hip: geometry collision cylinder length=0.05 radius=0.07; visual mesh filename=package://b2_driver_description/meshes/RL_hip.dae
- link RL_thigh: geometry collision box size=0.25 0.028 0.04; visual mesh filename=package://b2_driver_description/meshes/RL_thigh.dae
- link RR_calf: geometry collision box size=0.05 0.028 0.035; collision box size=0.1 0.0245 0.018
- link RR_hip: geometry collision cylinder length=0.05 radius=0.07; visual mesh filename=package://b2_driver_description/meshes/RR_hip.dae
- link RR_thigh: geometry collision box size=0.25 0.028 0.04; visual mesh filename=package://b2_driver_description/meshes/RR_thigh.dae
- link base_link: geometry collision box size=0.5 0.28 0.15; visual mesh filename=package://b2_driver_description/meshes/base_link.dae
